File: clock/clock.sch (KiCad schematic (older format))
At the start: 76 parts, among them J1 FTDI, J2 USB, J3 TP, SW1 SW_SPST, SW2 SW_SPST, SW3 SW_SPST, SW4 SW_SPST, SW5 SW_SPST, U1 iv12, U10 PCA9685PW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

Commit message: Changed USB footprint
Parts:
- J2: footprint Connector_USB:USB_Micro-B_Molex-105133-0001 -> Connector_USB:USB_Micro-B_Wuerth_614105150721_Vertical
Changed lines of the file:
@@
 F 0 "J2" H 1157 10167 50  0000 C CNN
 F 1 "USB" H 1157 10076 50  0000 C CNN
-F 2 "Connector_USB:USB_Micro-B_Molex-105133-0001" H 1250 9650 50  0001 C CNN
+F 2 "Connector_USB:USB_Micro-B_Wuerth_614105150721_Vertical" H 1250 9650 50  0001 C CNN
 F 3 "" H 1250 9650 50  0001 C CNN
 	1    1100 9700
