File: clock/_saved_clock.sch (KiCad schematic (older format))
At the start: 46 parts, among them J1 Conn_01x16_Male, J2 Conn_01x16_Male, U1 iv12, U2 iv12, U3 iv12, U4 iv12, U5 ULN2003, U6 ULN2003, U7 ULN2003, U8 ULN2003

Commit message: Rev 1 of clock display board
Parts:
- J3, J4, J5, J6: renamed from J?; footprint (none) -> Connector_PinHeader_2.54mm:PinHeader_1x01_P2.54mm_Vertical
- U1, U2, U3, U4: footprint tubes:iv12 -> tubes:iv12-large
Changed lines of the file:
@@
 F 0 "U2" H 2028 2353 60  0000 L CNN
 F 1 "iv12" H 2028 2247 60  0000 L CNN
-F 2 "tubes:iv12" H 1750 2300 60  0001 C CNN
+F 2 "tubes:iv12-large" H 1750 2300 60  0001 C CNN
 F 3 "" H 1750 2300 60  0001 C CNN
 	1    1750 2300
@@
 F 0 "U1" H 2028 4503 60  0000 L CNN
 F 1 "iv12" H 2028 4397 60  0000 L CNN
-F 2 "tubes:iv12" H 1750 4450 60  0001 C CNN
+F 2 "tubes:iv12-large" H 1750 4450 60  0001 C CNN
 F 3 "" H 1750 4450 60  0001 C CNN
 	1    1750 4450
@@
 F 0 "U3" H 10278 2453 60  0000 L CNN
 F 1 "iv12" H 10278 2347 60  0000 L CNN
-F 2 "tubes:iv12" H 10000 2400 60  0001 C CNN
+F 2 "tubes:iv12-large" H 10000 2400 60  0001 C CNN
 F 3 "" H 10000 2400 60  0001 C CNN
 	1    10000 2400
@@
 F 0 "U4" H 10278 4603 60  0000 L CNN
 F 1 "iv12" H 10278 4497 60  0000 L CNN
-F 2 "tubes:iv12" H 10000 4550 60  0001 C CNN
+F 2 "tubes:iv12-large" H 10000 4550 60  0001 C CNN
 F 3 "" H 10000 4550 60  0001 C CNN
 	1    10000 4550
@@
 	1850 3550 1850 3600
 $Comp
-L Connector:Conn_01x01_Male J?
+L Connector:Conn_01x01_Male J3
 U 1 1 5C37DF08
 P 2000 6900
-F 0 "J?" H 2108 7081 50  0000 C CNN
+F 0 "J3" H 2108 7081 50  0000 C CNN
 F 1 "Conn_01x01_Male" H 2108 6990 50  0000 C CNN
-F 2 "" H 2000 6900 50  0001 C CNN
+F 2 "Connector_PinHeader_2.54mm:PinHeader_1x01_P2.54mm_Vertical" H 2000 6900 50  0001 C CNN
 F 3 "~" H 2000 6900 50  0001 C CNN
 	1    2000 6900
@@
 $EndComp
 $Comp
-L Connector:Conn_01x01_Male J?
+L Connector:Conn_01x01_Male J4
 U 1 1 5C37E77F
 P 2000 7150
-F 0 "J?" H 2108 7331 50  0000 C CNN
+F 0 "J4" H 2108 7331 50  0000 C CNN
 F 1 "Conn_01x01_Male" H 2108 7240 50  0000 C CNN
-F 2 "" H 2000 7150 50  0001 C CNN
+F 2 "Connector_PinHeader_2.54mm:PinHeader_1x01_P2.54mm_Vertical" H 2000 7150 50  0001 C CNN
 F 3 "~" H 2000 7150 50  0001 C CNN
 	1    2000 7150
@@
 $EndComp
 $Comp
-L Connector:Conn_01x01_Male J?
+L Connector:Conn_01x01_Male J5
 U 1 1 5C37E94E
 P 3450 6850
-F 0 "J?" H 3422 6782 50  0000 R CNN
+F 0 "J5" H 3422 6782 50  0000 R CNN
 F 1 "Conn_01x01_Male" H 3422 6873 50  0000 R CNN
-F 2 "" H 3450 6850 50  0001 C CNN
+F 2 "Connector_PinHeader_2.54mm:PinHeader_1x01_P2.54mm_Vertical" H 3450 6850 50  0001 C CNN
 F 3 "~" H 3450 6850 50  0001 C CNN
 	1    3450 6850
@@
 $EndComp
 $Comp
-L Connector:Conn_01x01_Male J?
+L Connector:Conn_01x01_Male J6
 U 1 1 5C37EA85
 P 3450 7100
-F 0 "J?" H 3422 7032 50  0000 R CNN
+F 0 "J6" H 3422 7032 50  0000 R CNN
 F 1 "Conn_01x01_Male" H 3422 7123 50  0000 R CNN
-F 2 "" H 3450 7100 50  0001 C CNN
+F 2 "Connector_PinHeader_2.54mm:PinHeader_1x01_P2.54mm_Vertical" H 3450 7100 50  0001 C CNN
 F 3 "~" H 3450 7100 50  0001 C CNN
 	1    3450 7100
@@
 $EndComp
 $Comp
-L power:GND #PWR?
+L power:GND #PWR0123
 U 1 1 5C37ED87
 P 2300 7250
-F 0 "#PWR?" H 2300 7000 50  0001 C CNN
+F 0 "#PWR0123" H 2300 7000 50  0001 C CNN
 F 1 "GND" H 2305 7077 50  0000 C CNN
 F 2 "" H 2300 7250 50  0001 C CNN
@@
 	2300 7150 2300 7250
 $Comp
-L power:GND #PWR?
+L power:GND #PWR0124
 U 1 1 5C391947
 P 3150 7200
-F 0 "#PWR?" H 3150 6950 50  0001 C CNN
+F 0 "#PWR0124" H 3150 6950 50  0001 C CNN
 F 1 "GND" H 3155 7027 50  0000 C CNN
 F 2 "" H 3150 7200 50  0001 C CNN
@@
 	3150 7100 3250 7100
 $Comp
-L power:+5V #PWR?
+L power:+5V #PWR0125
 U 1 1 5C3A4B4D
 P 2300 6750
-F 0 "#PWR?" H 2300 6600 50  0001 C CNN
+F 0 "#PWR0125" H 2300 6600 50  0001 C CNN
 F 1 "+5V" H 2315 6923 50  0000 C CNN
 F 2 "" H 2300 6750 50  0001 C CNN
@@
 	3150 6850 3250 6850
 $Comp
-L power:+24V #PWR?
+L power:+24V #PWR0126
 U 1 1 5C3CC94C
 P 3150 6750
-F 0 "#PWR?" H 3150 6600 50  0001 C CNN
+F 0 "#PWR0126" H 3150 6600 50  0001 C CNN
 F 1 "+24V" H 3165 6923 50  0000 C CNN
 F 2 "" H 3150 6750 50  0001 C CNN
