File: iv12.sch (KiCad schematic (older format))
At the start: 4 parts, among them J1 CONN_01X08, J2 CONN_01X01, J3 CONN_01X01, U1 iv12

Commit message: Files missed from last commit.
Parts:
- J1: symbol CONN_01X08 -> conn1:CONN_01X08
- J2, J3: symbol CONN_01X01 -> conn1:CONN_01X01
- U1: footprint tubes:iv12 -> tubes:iv12-large; symbol iv12 -> iv12-rescue:iv12-RESCUE-iv12
Connections:
- net +1V5: now also J3.1 (P1); no longer J2.1 (P1)
- net +24V: now also J1.1 (P1); no longer J3.1 (P1)
- net GND: now also J2.1 (P1); no longer J1.1 (P1)
Other:
- moved on the sheet: J2, J3
Changed lines of the file:
@@
-EESchema Schematic File Version 3
-LIBS:power
-LIBS:device
-LIBS:transistors
-LIBS:conn
-LIBS:linear
-LIBS:regul
-LIBS:74xx
-LIBS:cmos4000
-LIBS:adc-dac
-LIBS:memory
-LIBS:xilinx
-LIBS:microcontrollers
-LIBS:dsp
-LIBS:microchip
-LIBS:analog_switches
-LIBS:motorola
-LIBS:texas
-LIBS:intel
-LIBS:audio
-LIBS:interface
-LIBS:digital-audio
-LIBS:philips
-LIBS:display
-LIBS:cypress
-LIBS:siliconi
-LIBS:opto
-LIBS:atmel
-LIBS:contrib
-LIBS:valves
-LIBS:iv12
+EESchema Schematic File Version 4
+LIBS:iv12-cache
 EELAYER 26 0
 EELAYER END
@@
 $EndDescr
 $Comp
-L CONN_01X08 J1
+L conn1:CONN_01X08 J1
 U 1 1 5A8F5D16
 P 5200 4050
@@
 $EndComp
 $Comp
-L CONN_01X01 J2
+L conn1:CONN_01X01 J2
 U 1 1 5A8F5D69
+P 6400 4400
+F 0 "J2" V 6450 4250 50  0000 R CNN
+F 1 "CONN_01X01" V 6350 4250 50  0000 R CNN
+F 2 "Pin_Headers:Pin_Header_Straight_1x01_Pitch2.54mm" H 6400 4400 50  0001 C CNN
+F 3 "" H 6400 4400 50  0001 C CNN
+	1    6400 4400
+	0    -1   -1   0
+$EndComp
+$Comp
+L conn1:CONN_01X01 J3
+U 1 1 5A8F5E1D
 P 5650 3100
-F 0 "J2" V 5650 3300 50  0000 R CNN
-F 1 "CONN_01X01" V 5550 3700 50  0000 R CNN
+F 0 "J3" V 5700 3300 50  0000 R CNN
+F 1 "CONN_01X01" V 5600 3700 50  0000 R CNN
 F 2 "Pin_Headers:Pin_Header_Straight_1x01_Pitch2.54mm" H 5650 3100 50  0001 C CNN
 F 3 "" H 5650 3100 50  0001 C CNN
 	1    5650 3100
-	0    -1   -1   0
-$EndComp
-$Comp
-L CONN_01X01 J3
-U 1 1 5A8F5E1D
-P 6350 3100
-F 0 "J3" V 6350 3000 50  0000 R CNN
-F 1 "CONN_01X01" V 6250 3000 50  0000 R CNN
-F 2 "Pin_Headers:Pin_Header_Straight_1x01_Pitch2.54mm" H 6350 3100 50  0001 C CNN
-F 3 "" H 6350 3100 50  0001 C CNN
-	1    6350 3100
 	0    -1   -1   0
 $EndComp
@@
 Wire Wire Line
 	5550 4300 5400 4300
-Wire Wire Line
-	5400 4400 5450 4400
-Wire Wire Line
-	5450 4400 5450 4650
-Wire Wire Line
-	5450 4650 6000 4650
-Wire Wire Line
-	6000 4600 6000 4750
 $Comp
-L iv12 U1
+L iv12-rescue:iv12-RESCUE-iv12 U1
 U 1 1 5A8F5C42
 P 6000 4000
 F 0 "U1" H 6050 4100 60  0000 R CNN
 F 1 "iv12" H 6100 4000 60  0000 R CNN
-F 2 "tubes:iv12" H 6000 4000 60  0001 C CNN
+F 2 "tubes:iv12-large" H 6000 4000 60  0001 C CNN
 F 3 "" H 6000 4000 60  0001 C CNN
 	1    6000 4000
@@
 $EndComp
 Wire Wire Line
-	5900 3200 5900 3400
-Wire Wire Line
-	6100 3200 6100 3400
+	5900 3200 5900 3300
 $Comp
-L GND #PWR?
+L power1:GND #PWR0101
 U 1 1 5A8F65FE
 P 6000 4750
-F 0 "#PWR?" H 6000 4500 50  0001 C CNN
+F 0 "#PWR0101" H 6000 4500 50  0001 C CNN
 F 1 "GND" H 6005 4577 50  0000 C CNN
 F 2 "" H 6000 4750 50  0001 C CNN
@@
 	1    0    0    -1
 $EndComp
-Connection ~ 6000 4650
 $Comp
-L +24V #PWR?
+L power1:+24V #PWR0102
 U 1 1 5A8F66BE
 P 6100 3200
-F 0 "#PWR?" H 6100 3050 50  0001 C CNN
+F 0 "#PWR0102" H 6100 3050 50  0001 C CNN
 F 1 "+24V" H 6115 3373 50  0000 C CNN
 F 2 "" H 6100 3200 50  0001 C CNN
@@
 	1    0    0    -1
 $EndComp
-Wire Wire Line
-	6350 3300 6100 3300
-Connection ~ 6100 3300
 $Comp
-L +1V5 #PWR?
+L power1:+1V5 #PWR0103
 U 1 1 5A8F67D0
 P 5900 3200
-F 0 "#PWR?" H 5900 3050 50  0001 C CNN
+F 0 "#PWR0103" H 5900 3050 50  0001 C CNN
 F 1 "+1V5" H 5915 3373 50  0000 C CNN
 F 2 "" H 5900 3200 50  0001 C CNN
@@
 	5900 3300 5650 3300
 Connection ~ 5900 3300
+Wire Wire Line
+	5900 3300 5900 3400
+Wire Wire Line
+	6000 4600 6000 4650
+$Comp
+L power1:+24V #PWR0104
+U 1 1 5AAAFBE7
+P 5550 4500
+F 0 "#PWR0104" H 5550 4350 50  0001 C CNN
+F 1 "+24V" H 5565 4673 50  0000 C CNN
+F 2 "" H 5550 4500 50  0001 C CNN
+F 3 "" H 5550 4500 50  0001 C CNN
+	1    5550 4500
+	1    0    0    -1
+$EndComp
+Wire Wire Line
+	5400 4400 5450 4400
+Wire Wire Line
+	5450 4400 5450 4600
+Wire Wire Line
+	5450 4600 5550 4600
+Wire Wire Line
+	5550 4600 5550 4500
+Wire Wire Line
+	6000 4650 6400 4650
+Wire Wire Line
+	6400 4650 6400 4600
+Connection ~ 6000 4650
+Wire Wire Line
+	6000 4650 6000 4750
+Wire Wire Line
+	6100 3200 6100 3400
 $EndSCHEMATC
