File: iv12.kicad_pcb (KiCad board)
At the start: 2 copper layers, 20.3 x 25.4 mm, 5 parts, among them J1 CONN_01X08, J2 CONN_01X01, J3 CONN_01X01, U1 iv12

Commit message: Files missed from last commit.
Parts:
- U1: footprint tubes:iv12 -> tubes:iv12-large
- moved J1 17.8 mm to (156.2, 96.5), turned to 270 degrees
- turned J2 to 270 degrees
Connections:
- J1 pad 1: GND -> +24V
- J2 pad 1: +1V5 -> GND
- J3 pad 1: +24V -> +1V5
Routing:
- net Net-(J1-Pad8): track 31.1 -> 14.3 mm
- net +24V: track 10.4 -> 21.8 mm
- net Net-(J1-Pad6): track 11.8 -> 22.7 mm
- net Net-(J1-Pad5): track 17.3 -> 24.7 mm
- net Net-(J1-Pad3): track 10.1 -> 16.5 mm
- net Net-(J1-Pad4): track 19.2 -> 23.4 mm
- net Net-(J1-Pad2): track 18.0 -> 14.1 mm
- net Net-(J1-Pad7): track 19.5 -> 16.4 mm
- net +1V5: track 13.9 -> 12.5 mm
Other:
- board text added: "F+"
- board text added: "F-"
- board text added: "G+"
- board text added: "Rev. 2"
- board text removed: "HV"
- board text removed: "LV"
- board text removed: "Rev. 1"

Commit message: Made labels for segments lowercase to reduce confusion it G and G+
Other:
- board text added: "a"
- board text added: "b"
- board text added: "c"
- board text added: "d"
- board text added: "e"
- board text added: "f"
- board text added: "g"
- board text removed: "A"
- board text removed: "B"
- board text removed: "C"
- board text removed: "D"
- board text removed: "E"
- board text removed: "F"
- board text removed: "G"
Changed lines of the file:
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@@
     (effects (font (size 1 1) (thickness 0.2)))
   )
-  (gr_text E (at 148.59 98.552) (layer F.SilkS)
+  (gr_text e (at 148.59 98.552) (layer F.SilkS)
     (effects (font (size 1 1) (thickness 0.2)))
   )
@@
     (effects (font (size 1 1) (thickness 0.2)))
   )
-  (gr_text A (at 138.43 98.552) (layer F.SilkS)
+  (gr_text a (at 138.43 98.552) (layer F.SilkS)
     (effects (font (size 1 1) (thickness 0.2)))
   )
@@
     (effects (font (size 1 1) (thickness 0.2)))
   )
-  (gr_text G (at 153.67 98.552) (layer F.SilkS)
+  (gr_text g (at 153.67 98.552) (layer F.SilkS)
     (effects (font (size 1 1) (thickness 0.2)))
   )
-  (gr_text F (at 151.13 98.552) (layer F.SilkS)
+  (gr_text f (at 151.13 98.552) (layer F.SilkS)
     (effects (font (size 1 1) (thickness 0.2)))
   )
-  (gr_text D (at 146.05 98.552) (layer F.SilkS)
+  (gr_text d (at 146.05 98.552) (layer F.SilkS)
     (effects (font (size 1 1) (thickness 0.2)))
   )
-  (gr_text C (at 143.51 98.552) (layer F.SilkS)
+  (gr_text c (at 143.51 98.552) (layer F.SilkS)
     (effects (font (size 1 1) (thickness 0.2)))
   )
-  (gr_text B (at 140.97 98.552) (layer F.SilkS)
+  (gr_text b (at 140.97 98.552) (layer F.SilkS)
     (effects (font (size 1 1) (thickness 0.2)))
   )
